Commit message: il robot si muove ma non perfettamente

File: ros2_fra2mo/urdf/fra2mo.urdf.xacro (robot description, xacro)
@@ -3,4 +3,5 @@
   <xacro:include filename="$(find ros2_fra2mo)/urdf/fra2mo_base_macro.xacro"/>
   <xacro:include filename="$(find ros2_fra2mo)/urdf/lidar_gazebo_macro.xacro"/>
+  <xacro:include filename="$(find ros2_fra2mo)/urdf/trailer_macro.xacro"/>
   <!-- <xacro:include filename="$(find ros2_fra2mo)/urdf/d435_gazebo_macro.xacro" />  -->
   <xacro:property name="LIDAR" value="True"/>
@@ -8,4 +9,6 @@
   <!-- Diff Drive Robot Base -->
   <xacro:fra2mo_base/>
+  <!-- Cassone trainato -->
+  <xacro:fra2mo_trailer parent_link="base_link"/>
   <!-- LIDAR Sensor-->
   <xacro:if value="${LIDAR}">

File: ros2_fra2mo/urdf/lidar_gazebo_macro.xacro (robot description, xacro)
@@ -38,6 +38,6 @@
                       <samples>640</samples>
                       <resolution>1</resolution>
-                      <min_angle>-3.14</min_angle>
-                      <max_angle>3.14</max_angle>
+                      <min_angle>-1.57</min_angle>
+                      <max_angle>1.57</max_angle>
                   </horizontal>
                   <!--<vertical>

File: ros2_iiwa/iiwa_description/urdf/iiwa.urdf.xacro (robot description, xacro)
@@ -2,227 +2,335 @@
 <robot xmlns:xacro="http://www.ros.org/wiki/xacro">
   <xacro:macro name="iiwa" params="parent prefix *origin">
-  <material name="gray">
-    <color rgba="0.5 0.5 0.5 1.0"/>
-  </material>
-  <link name="${prefix}iiwa_base" type="fixed"/>
-  <joint name="${prefix}iiwa_root_joint" type="fixed">
-      <xacro:insert_block name="origin" />
-      <parent link="${parent}"/>
-      <child link="${prefix}iiwa_base"/>
-  </joint>
-  <joint name="${prefix}iiwa_base_joint" type="fixed">
-      <origin rpy="0.0 0 0" xyz="0 0 0"/>
-      <parent link="${prefix}iiwa_base"/>
-      <child link="${prefix}link_0"/>
-  </joint>
-  <link name="${prefix}link_0">
+    <material name="gray">
+      <color rgba="0.5 0.5 0.5 1.0"/>
+    </material>
+    <link name="${prefix}iiwa_base" type="fixed"/>
+    <joint name="${prefix}iiwa_root_joint" type="fixed">
+        <xacro:insert_block name="origin" />
+        <parent link="${parent}"/>
+        <child link="${prefix}iiwa_base"/>
+    </joint>
+    <joint name="${prefix}iiwa_base_joint" type="fixed">
+        <origin rpy="0.0 0 0" xyz="0 0 0"/>
+        <parent link="${prefix}iiwa_base"/>
+        <child link="${prefix}link_0"/>
+    </joint>
+    <link name="${prefix}link_0">
+        <visual>
+          <origin rpy="0.0 0 0" xyz="0 0 0"/>
+          <geometry>
+            <mesh filename="file://$(find iiwa_description)/meshes/lbr_iiwa_14_r820/visual/base_link.dae"/>
+          </geometry>
+        </visual>
+        <collision>
+          <origin rpy="0 0 0" xyz="0 0 0"/>
+          <geometry>
+            <mesh filename="file://$(find iiwa_description)/meshes/lbr_iiwa_14_r820/collision/base_link.stl"/>
+          </geometry>
+        </collision>
+        <inertial>
+          <origin xyz="-0.1 0 0.07" rpy="0 0 0"/>
+          <mass value="5"/>
+          <inertia ixx="0.05"  ixy="0"  ixz="0" iyy="0.06" iyz="0" izz="0.03" />
+        </inertial>
+    </link>
+    <link name="${prefix}link_1">
+        <visual>
+          <origin rpy="0 0 0" xyz="0 0 0"/>
+          <geometry>
+            <mesh filename="file://$(find iiwa_description)/meshes/lbr_iiwa_14_r820/visual/link_1.dae"/>
+          </geometry>
+        </visual>
+        <collision>
+          <origin rpy="0 0 0" xyz="0 0 0"/>
+          <geometry>
+            <mesh filename="file://$(find iiwa_description)/meshes/lbr_iiwa_14_r820/collision/link_1.stl"/>
+          </geometry>
+        </collision>
+        <inertial>
+          <origin xyz="0 -0.03 0.12" rpy="0 0 0"/>
+          <mass value="4"/>
+          <inertia ixx="0.1"  ixy="0"  ixz="0" iyy="0.09" iyz="0" izz="0.02" />
+        </inertial>
+    </link>
+    <link name="${prefix}link_2">
+        <visual>
+          <origin rpy="0 0 0" xyz="0 0 0"/>
+          <geometry>
+            <mesh filename="file://$(find iiwa_description)/meshes/lbr_iiwa_14_r820/visual/link_2.dae"/>
+          </geometry>
+        </visual>
+        <collision>
+          <origin rpy="0 0 0" xyz="0 0 0"/>
+          <geometry>
+            <mesh filename="file://$(find iiwa_description)/meshes/lbr_iiwa_14_r820/collision/link_2.stl"/>
+          </geometry>
+        </collision>
+        <inertial>
+          <origin xyz="0.0003 0.059 0.042" rpy="0 0 0"/>
+          <mass value="4"/>
+          <inertia ixx="0.05"  ixy="0"  ixz="0" iyy="0.018" iyz="0" izz="0.044" />
+        </inertial>
+    </link>
+    <link name="${prefix}link_3">
+        <visual>
+          <origin rpy="0 0 0" xyz="0 0 0"/>
+          <geometry>
+            <mesh filename="file://$(find iiwa_description)/meshes/lbr_iiwa_14_r820/visual/link_3.dae"/>
+          </geometry>
+        </visual>
+        <collision>
+          <origin rpy="0 0 0" xyz="0 0 0"/>
+          <geometry>
+            <mesh filename="file://$(find iiwa_description)/meshes/lbr_iiwa_14_r820/collision/link_3.stl"/>
+          </geometry>
+        </collision>
+        <inertial>
+          <origin xyz="0 0.03 0.13" rpy="0 0 0"/>
+          <mass value="3"/>
+          <inertia ixx="0.08"  ixy="0"  ixz="0" iyy="0.075" iyz="0" izz="0.01" />
+        </inertial>
+    </link>
+    <link name="${prefix}link_4">
+        <visual>
+          <origin rpy="0 0 0" xyz="0 0 0"/>
+          <geometry>
+            <mesh filename="file://$(find iiwa_description)/meshes/lbr_iiwa_14_r820/visual/link_4.dae"/>
+          </geometry>
+        </visual>
+        <collision>
+          <origin rpy="0 0 0" xyz="0 0 0"/>
+          <geometry>
+            <mesh filename="file://$(find iiwa_description)/meshes/lbr_iiwa_14_r820/collision/link_4.stl"/>
+          </geometry>
+        </collision>
+        <inertial>
+          <origin xyz="0 0.067 0.034" rpy="0 0 0"/>
+          <mass value="2.7"/>
+          <inertia ixx="0.03"  ixy="0"  ixz="0" iyy="0.01" iyz="0" izz="0.029" />
+        </inertial>
+    </link>
+    <link name="${prefix}link_5">
+        <visual>
+          <origin rpy="0 0 0" xyz="0 0 0"/>
+          <geometry>
+            <mesh filename="file://$(find iiwa_description)/meshes/lbr_iiwa_14_r820/visual/link_5.dae"/>
+          </geometry>
+        </visual>
+        <collision>
+          <origin rpy="0 0 0" xyz="0 0 0"/>
+          <geometry>
+            <mesh filename="file://$(find iiwa_description)/meshes/lbr_iiwa_14_r820/collision/link_5.stl"/>
+          </geometry>
+        </collision>
+        <inertial>
+          <origin xyz="0.0001 0.021 0.076" rpy="0 0 0"/>
+          <mass value="1.7"/>
+          <inertia ixx="0.02"  ixy="0"  ixz="0" iyy="0.018" iyz="0" izz="0.005" />
+        </inertial>
+    </link>
+    <link name="${prefix}link_6">
+        <visual>
+          <origin rpy="0 0 0" xyz="0 0 0"/>
+          <geometry>
+            <mesh filename="file://$(find iiwa_description)/meshes/lbr_iiwa_14_r820/visual/link_6.dae"/>
+          </geometry>
+        </visual>
+        <collision>
+          <origin rpy="0 0 0" xyz="0 0 0"/>
+          <geometry>
+            <mesh filename="file://$(find iiwa_description)/meshes/lbr_iiwa_14_r820/collision/link_6.stl"/>
+          </geometry>
+        </collision>
+        <inertial>
+          <origin xyz="0 0.0006 0.0004" rpy="0 0 0"/>
+          <mass value="1.8"/>
+          <inertia ixx="0.025"  ixy="0"  ixz="0" iyy="0.0136" iyz="0" izz="0.0247" />
+        </inertial>
+    </link>
+    <link name="${prefix}link_7">
+        <visual>
+          <origin rpy="0 0 0" xyz="0 0 0.07"/>
+          <material name="gray"/>
+          <geometry>
+            <mesh filename="file://$(find iiwa_description)/meshes/lbr_iiwa_14_r820/visual/link_7_2.stl" scale ="0.001 0.001 0.001"/>
+          </geometry>
+        </visual>
+        <collision>
+          <origin rpy="0 0 0" xyz="0 0 0.07"/>
+          <geometry>
+            <mesh filename="file://$(find iiwa_description)/meshes/lbr_iiwa_14_r820/collision/link_7_2.stl" scale ="0.001 0.001 0.001"/>
+          </geometry>
+        </collision>
+        <inertial>
+          <origin xyz="0 0 0.02" rpy="0 0 0"/>
+          <mass value="${0.3 / 0.308 * 0.44}"/>
+          <inertia ixx="0.01"  ixy="0"  ixz="0" iyy="0.01" iyz="0" izz="0.01" />
+        </inertial>
+    </link>
+    <link name="${prefix}tool0"/>
+    <joint name="${prefix}joint_a1" type="revolute">
+        <origin rpy="0 0 0" xyz="0 0 0"/>
+        <parent link="${prefix}link_0"/>
+        <child link="${prefix}link_1"/>
+        <axis xyz="0 0 1"/>
+        <limit effort="320" lower="-2.9668" upper="2.9668" velocity="1.4834"/>
+    </joint>
+    <joint name="${prefix}joint_a2" type="revolute">
+        <origin rpy="0 0 0" xyz="-0.00043624 0 0.36"/>
+        <parent link="${prefix}link_1"/>
+        <child link="${prefix}link_2"/>
+        <axis xyz="0 1 0"/>
+        <limit effort="320" lower="-2.0942" upper="2.0942" velocity="1.4834"/>
+    </joint>
+    <joint name="${prefix}joint_a3" type="revolute">
+        <origin rpy="0 0 0" xyz="0 0 0"/>
+        <parent link="${prefix}link_2"/>
+        <child link="${prefix}link_3"/>
+        <axis xyz="0 0 1"/>
+        <limit effort="176" lower="-2.9668" upper="2.9668" velocity="1.7452"/>
+    </joint>
+    <joint name="${prefix}joint_a4" type="revolute">
+        <origin rpy="0 0 0" xyz="0.00043624 0 0.42"/>
+        <parent link="${prefix}link_3"/>
+        <child link="${prefix}link_4"/>
+        <axis xyz="0 -1 0"/>
+        <limit effort="176" lower="-2.0942" upper="2.0942" velocity="1.3089"/>
+    </joint>
+    <joint name="${prefix}joint_a5" type="revolute">
+        <origin rpy="0 0 0" xyz="0 0 0"/>
+        <parent link="${prefix}link_4"/>
+        <child link="${prefix}link_5"/>
+        <axis xyz="0 0 1"/>
+        <limit effort="110" lower="-2.9668" upper="2.9668" velocity="2.2688"/>
+    </joint>
+    <joint name="${prefix}joint_a6" type="revolute">
+        <origin rpy="0 0 0" xyz="0 0 0.4"/>
+        <parent link="${prefix}link_5"/>
+        <child link="${prefix}link_6"/>
+        <axis xyz="0 1 0"/>
+        <limit effort="40" lower="-2.0942" upper="2.0942" velocity="2.356"/>
+    </joint>
+    <joint name="${prefix}joint_a7" type="revolute">
+        <origin rpy="0 0 0" xyz="0 0 0"/>
+        <parent link="${prefix}link_6"/>
+        <child link="${prefix}link_7"/>
+        <axis xyz="0 0 1"/>
+        <limit effort="40" lower="-3.0541" upper="3.0541" velocity="2.356"/>
+    </joint>
+    <joint name="${prefix}joint_a7-tool0" type="fixed">
+        <origin rpy="0 0 0" xyz="0 0 0.154"/>
+        <parent link="${prefix}link_7"/>
+        <child link="${prefix}tool0"/>
+        <axis xyz="0 0 0"/>
+    </joint>
+    <joint name="${prefix}camera_joint" type="fixed">
+        <parent link="${prefix}tool0"/>
+        <child link="${prefix}camera_link"/>
+        <origin xyz="0.07 0.0 -0.03" rpy="3.14 -1.57 0"/>
+    </joint>
+    <link name="${prefix}camera_link">
+        <visual>
+          <geometry>
+            <box size="0.03 0.03 0.03"/>
+          </geometry>
+          <material name="black">
+            <color rgba="0 0 0 1"/>
+          </material>
+        </visual>
+        <collision>
+          <geometry>
+            <box size="0.03 0.03 0.03"/>
+          </geometry>
+        </collision>
+        <inertial>
+          <mass value="0.05"/>
+          <inertia ixx="0.0001" ixy="0" ixz="0" iyy="0.0001" iyz="0" izz="0.0001"/>
+        </inertial>
+    </link>
+    <joint name="${prefix}camera_optical_joint" type="fixed">
+        <parent link="${prefix}camera_link"/>
+        <child link="${prefix}camera_optical_frame"/>
+        <origin xyz="0 0 0" rpy="-1.5708 0 -1.5708"/>
+    </joint>
+    <link name="${prefix}camera_optical_frame"/>
+    <link name="${prefix}vacuum_gripper_link">
       <visual>
-        <origin rpy="0.0 0 0" xyz="0 0 0"/>
         <geometry>
-          <mesh filename="file://$(find iiwa_description)/meshes/lbr_iiwa_14_r820/visual/base_link.dae"/>
+          <cylinder radius="0.04" length="0.02"/>
         </geometry>
+        <material name="Black">
+          <color rgba="0.1 0.1 0.1 1"/>
+        </material>
+        <origin xyz="0 0 0.01" rpy="0 0 0"/>
       </visual>
-      <collision>
-        <origin rpy="0 0 0" xyz="0 0 0"/>
+      <collision name="${prefix}vacuum_gripper_collision">
         <geometry>
-          <mesh filename="file://$(find iiwa_description)/meshes/lbr_iiwa_14_r820/collision/base_link.stl"/>
+          <cylinder radius="0.04" length="0.02"/>
         </geometry>
+        <origin xyz="0 0 0.01" rpy="0 0 0"/>
       </collision>
       <inertial>
-        <origin xyz="-0.1 0 0.07" rpy="0 0 0"/>
-        <mass value="5"/>
-        <inertia ixx="0.05"  ixy="0"  ixz="0" iyy="0.06" iyz="0" izz="0.03" />
+        <mass value="0.1"/>
+        <inertia ixx="0.0001" ixy="0" ixz="0" iyy="0.0001" iyz="0" izz="0.0001"/>
       </inertial>
-  </link>
-  <link name="${prefix}link_1">
-      <visual>
-        <origin rpy="0 0 0" xyz="0 0 0"/>
-        <geometry>
-          <mesh filename="file://$(find iiwa_description)/meshes/lbr_iiwa_14_r820/visual/link_1.dae"/>
-        </geometry>
-      </visual>
-      <collision>
-        <origin rpy="0 0 0" xyz="0 0 0"/>
-        <geometry>
-          <mesh filename="file://$(find iiwa_description)/meshes/lbr_iiwa_14_r820/collision/link_1.stl"/>
-        </geometry>
-      </collision>
-      <inertial>
-        <origin xyz="0 -0.03 0.12" rpy="0 0 0"/>
-        <mass value="4"/>
-        <inertia ixx="0.1"  ixy="0"  ixz="0" iyy="0.09" iyz="0" izz="0.02" />
-      </inertial>
-  </link>
-  <link name="${prefix}link_2">
-      <visual>
-        <origin rpy="0 0 0" xyz="0 0 0"/>
-        <geometry>
-          <mesh filename="file://$(find iiwa_description)/meshes/lbr_iiwa_14_r820/visual/link_2.dae"/>
-        </geometry>
-      </visual>
-      <collision>
-        <origin rpy="0 0 0" xyz="0 0 0"/>
-        <geometry>
-          <mesh filename="file://$(find iiwa_description)/meshes/lbr_iiwa_14_r820/collision/link_2.stl"/>
-        </geometry>
-      </collision>
-      <inertial>
-        <origin xyz="0.0003 0.059 0.042" rpy="0 0 0"/>
-        <mass value="4"/>
-        <inertia ixx="0.05"  ixy="0"  ixz="0" iyy="0.018" iyz="0" izz="0.044" />
-      </inertial>
-  </link>
-  <link name="${prefix}link_3">
-      <visual>
-        <origin rpy="0 0 0" xyz="0 0 0"/>
-        <geometry>
-          <mesh filename="file://$(find iiwa_description)/meshes/lbr_iiwa_14_r820/visual/link_3.dae"/>
-        </geometry>
-      </visual>
-      <collision>
-        <origin rpy="0 0 0" xyz="0 0 0"/>
-        <geometry>
-          <mesh filename="file://$(find iiwa_description)/meshes/lbr_iiwa_14_r820/collision/link_3.stl"/>
-        </geometry>
-      </collision>
-      <inertial>
-        <origin xyz="0 0.03 0.13" rpy="0 0 0"/>
-        <mass value="3"/>
-        <inertia ixx="0.08"  ixy="0"  ixz="0" iyy="0.075" iyz="0" izz="0.01" />
-      </inertial>
-  </link>
-  <link name="${prefix}link_4">
-      <visual>
-        <origin rpy="0 0 0" xyz="0 0 0"/>
-        <geometry>
-          <mesh filename="file://$(find iiwa_description)/meshes/lbr_iiwa_14_r820/visual/link_4.dae"/>
-        </geometry>
-      </visual>
-      <collision>
-        <origin rpy="0 0 0" xyz="0 0 0"/>
-        <geometry>
-          <mesh filename="file://$(find iiwa_description)/meshes/lbr_iiwa_14_r820/collision/link_4.stl"/>
-        </geometry>
-      </collision>
-      <inertial>
-        <origin xyz="0 0.067 0.034" rpy="0 0 0"/>
-        <mass value="2.7"/>
-        <inertia ixx="0.03"  ixy="0"  ixz="0" iyy="0.01" iyz="0" izz="0.029" />
-      </inertial>
-  </link>
-  <link name="${prefix}link_5">
-      <visual>
-        <origin rpy="0 0 0" xyz="0 0 0"/>
-        <geometry>
-          <mesh filename="file://$(find iiwa_description)/meshes/lbr_iiwa_14_r820/visual/link_5.dae"/>
-        </geometry>
-      </visual>
-      <collision>
-        <origin rpy="0 0 0" xyz="0 0 0"/>
-        <geometry>
-          <mesh filename="file://$(find iiwa_description)/meshes/lbr_iiwa_14_r820/collision/link_5.stl"/>
-        </geometry>
-      </collision>
-      <inertial>
-        <origin xyz="0.0001 0.021 0.076" rpy="0 0 0"/>
-        <mass value="1.7"/>
-        <inertia ixx="0.02"  ixy="0"  ixz="0" iyy="0.018" iyz="0" izz="0.005" />
-      </inertial>
-  </link>
-  <link name="${prefix}link_6">
-      <visual>
-        <origin rpy="0 0 0" xyz="0 0 0"/>
-        <geometry>
-          <mesh filename="file://$(find iiwa_description)/meshes/lbr_iiwa_14_r820/visual/link_6.dae"/>
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