Commit message: modifica della macchina a stati 2/totale

File: ros2_iiwa/iiwa_description/gazebo/iiwa.gazebo.xacro (robot description, xacro)
@@ -13,6 +13,6 @@
     <!-- Camera sensor plugin per Ignition Gazebo -->
     <gazebo reference="${prefix}camera_link">
-        <sensor name="${prefix}camera" type="camera">
-            <camera name="iiwa_camera">
+        <sensor name="camera" type="camera">
+            <camera>
                 <horizontal_fov>1.047</horizontal_fov>
                 <image>
@@ -25,4 +25,9 @@
                     <far>100</far>
                 </clip>
+                <noise>
+                    <type>gaussian</type>
+                    <mean>0.0</mean>
+                    <stddev>0.007</stddev>
+                </noise>
             </camera>
             <always_on>1</always_on>
@@ -32,25 +37,4 @@
         </sensor>
     </gazebo>
-    <!-- Camera info publisher per Ignition Gazebo -->
-    <gazebo reference="${prefix}camera_link">
-        <sensor name="${prefix}camera_info" type="camera">
-            <camera name="iiwa_camera_info">
-                <horizontal_fov>1.047</horizontal_fov>
-                <image>
-                    <width>640</width>
-                    <height>480</height>
-                    <format>RGB_INT8</format>
-                </image>
-                <clip>
-                    <near>0.01</near>
-                    <far>100</far>
-                </clip>
-            </camera>
-            <always_on>1</always_on>
-            <update_rate>30</update_rate>
-            <visualize>false</visualize>
-            <topic>camera/camera_info</topic>
-        </sensor>
-    </gazebo>
   </xacro:macro>
 </robot>

File: ros2_iiwa/iiwa_description/urdf/iiwa.urdf.xacro (robot description, xacro)
@@ -228,5 +228,5 @@
         <parent link="${prefix}tool0"/>
         <child link="${prefix}camera_link"/>
-        <origin xyz="0.07 0.0 -0.03" rpy="3.14 -1.57 0"/>
+        <origin xyz="-0.07 0.0 -0.03" rpy="3.14 -1.57 0"/>
     </joint>
     <link name="${prefix}camera_link">
